File: original/power supply.sch (KiCad schematic (older format))
At the start: 8 parts, among them J1 Conn_IEC_Power, T2 PwrTxfmr

Commit message: adding some components to try to stop a high pitch squal sound I sometimes hear from the amp
Parts:
- J1: symbol local:Conn_IEC_Power -> nobsound-audio-amplifier-rescue:Conn_IEC_Power-local
- S1: symbol local:SW_SPST -> nobsound-audio-amplifier-rescue:SW_SPST-local
- T2: symbol local:PwrTxfmr -> nobsound-audio-amplifier-rescue:PwrTxfmr-local
- V3: symbol local:5Z4P -> nobsound-audio-amplifier-rescue:5Z4P-local
Changed lines of the file:
@@
 $EndDescr
 $Comp
-L local:5Z4P V3
+L nobsound-audio-amplifier-rescue:5Z4P-local V3
 U 1 1 5F152C6F
 P 6600 4000
@@
 $EndComp
 $Comp
-L local:PwrTxfmr T2
+L nobsound-audio-amplifier-rescue:PwrTxfmr-local T2
 U 1 1 5F15D5D5
 P 5300 4100
@@
 $EndComp
 $Comp
-L local:SW_SPST S1
+L nobsound-audio-amplifier-rescue:SW_SPST-local S1
 U 1 1 5F164E42
 P 4600 3800
@@
 $EndComp
 $Comp
-L local:Conn_IEC_Power J1
+L nobsound-audio-amplifier-rescue:Conn_IEC_Power-local J1
 U 1 1 5F1757DE
 P 3800 3900
