File: original/right_channel.sch (KiCad schematic (older format))
At the start: 20 parts, among them J4 Left 0 ohms, J5 Right 8 ohms, J6 Conn_Coaxial, T3 AudioTxfmr

Commit message: adding some components to try to stop a high pitch squal sound I sometimes hear from the amp
Parts:
- T3: symbol local:AudioTxfmr -> nobsound-audio-amplifier-rescue:AudioTxfmr-local
- V4,V5: symbol local:6P1 -> nobsound-audio-amplifier-rescue:6P1-local
- V7: symbol local:6H8C -> nobsound-audio-amplifier-rescue:6H8C-local
Connections:
- net Earth: now also C11.2, R?.1
- net at R13.1, V7.4 (g): now also C11.1; no longer C11.2
- net at C10.1, V4,V5.7 (g1): now also R?.2; no longer R?.1
Other:
- moved on the sheet: C11, R?
Changed lines of the file:
@@
 $EndDescr
 $Comp
-L local:AudioTxfmr T?
+L nobsound-audio-amplifier-rescue:AudioTxfmr-local T?
 U 1 1 5F20DF61
 P 7250 2250
@@
 Connection ~ 4200 1700
 $Comp
-L local:6H8C V?
+L nobsound-audio-amplifier-rescue:6H8C-local V?
 U 1 1 5F20DF83
 P 4700 2950
@@
 L Device:R R?
 U 1 1 5F20DF90
-P 4450 2400
+P 6400 3300
 AR Path="/5F20DF90" Ref="R?"  Part="1"
 AR Path="/5F1F04D2/5F20DF90" Ref="R?"  Part="1"
 AR Path="/5F200EB9/5F20DF90" Ref="R?"  Part="1"
-F 0 "R?" V 4243 2400 50  0000 C CNN
-F 1 "470K" V 4334 2400 50  0000 C CNN
-F 2 "" V 4380 2400 50  0001 C CNN
-F 3 "~" H 4450 2400 50  0001 C CNN
-	1    4450 2400
-	0    1    1    0
+F 0 "R?" V 6193 3300 50  0000 C CNN
+F 1 "470K" V 6284 3300 50  0000 C CNN
+F 2 "" V 6330 3300 50  0001 C CNN
+F 3 "~" H 6400 3300 50  0001 C CNN
+	1    6400 3300
+	-1   0    0    1
 $EndComp
 $Comp
 L Device:C C?
 U 1 1 5F20DF96
-P 4200 2750
+P 3950 3250
 AR Path="/5F20DF96" Ref="C?"  Part="1"
 AR Path="/5F1F04D2/5F20DF96" Ref="C?"  Part="1"
 AR Path="/5F200EB9/5F20DF96" Ref="C11"  Part="1"
-F 0 "C11" H 3750 2800 50  0000 L CNN
-F 1 "220K400" H 3750 2700 50  0000 L CNN
-F 2 "" H 4238 2600 50  0001 C CNN
-F 3 "~" H 4200 2750 50  0001 C CNN
-	1    4200 2750
+F 0 "C11" H 3500 3300 50  0000 L CNN
+F 1 "220K400" H 3500 3200 50  0000 L CNN
+F 2 "" H 3988 3100 50  0001 C CNN
+F 3 "~" H 3950 3250 50  0001 C CNN
+	1    3950 3250
 	1    0    0    -1
 $EndComp
@@
 $EndComp
 $Comp
-L local:6H8C V?
+L nobsound-audio-amplifier-rescue:6H8C-local V?
 U 2 1 5F20DFA3
 P 4700 4300
@@
 	4750 5750 5100 5750
 Wire Wire Line
-	4200 2900 4200 3000
-Wire Wire Line
 	4700 3850 4200 3850
 Connection ~ 4700 3850
 Wire Wire Line
 	4350 3000 4200 3000
-Connection ~ 4200 3000
 Wire Wire Line
 	4200 3000 4200 3100
-Wire Wire Line
-	5200 2200 5300 2200
-Wire Wire Line
-	4300 2400 4200 2400
-Wire Wire Line
-	4200 2400 4200 2600
-Wire Wire Line
-	4600 2400 5300 2400
-Wire Wire Line
-	5300 2400 5300 2200
-Connection ~ 5300 2200
-Wire Wire Line
-	5300 2200 5700 2200
 NoConn ~ 7550 2050
 $Comp
@@
 	7650 1850 7550 1850
 $Comp
-L local:6P1 V2,V?
+L nobsound-audio-amplifier-rescue:6P1-local V2,V?
 U 1 1 5F20E00F
 P 6950 2950
@@
 $EndComp
 Wire Wire Line
-	6600 3150 5700 3150
+	6600 3150 6400 3150
 Wire Wire Line
 	5700 3150 5700 2200
@@
 Wire Wire Line
 	3550 1700 3450 1700
+Wire Wire Line
+	5200 2200 5700 2200
+Connection ~ 6400 3150
+Wire Wire Line
+	6400 3150 5700 3150
+$Comp
+L power:Earth #PWR?
+U 1 1 5F61D356
+P 3950 3450
+F 0 "#PWR?" H 3950 3200 50  0001 C CNN
+F 1 "Earth" H 3950 3300 50  0001 C CNN
+F 2 "" H 3950 3450 50  0001 C CNN
+F 3 "~" H 3950 3450 50  0001 C CNN
+	1    3950 3450
+	1    0    0    -1
+$EndComp
+Wire Wire Line
+	3950 3450 3950 3400
+Wire Wire Line
+	3950 3100 3950 3000
+Wire Wire Line
+	3950 3000 4200 3000
+Connection ~ 4200 3000
+$Comp
+L power:Earth #PWR?
+U 1 1 5F620E36
+P 6400 3450
+F 0 "#PWR?" H 6400 3200 50  0001 C CNN
+F 1 "Earth" H 6400 3300 50  0001 C CNN
+F 2 "" H 6400 3450 50  0001 C CNN
+F 3 "~" H 6400 3450 50  0001 C CNN
+	1    6400 3450
+	1    0    0    -1
+$EndComp
 $EndSCHEMATC
