File: updated/left_channel.sch (KiCad schematic (older format))
At the start: 32 parts, among them J2 Left 8 ohms, J3 Left 0 ohms, J7 Conn_Coaxial, T1 AudioTxfmr

Commit message: It didn't sound right to me
I don't understand how changing the cathode bypass a bit made the amp a lot more brighter. Theory is the power supply was over loaded before and it was not able to drive the high frequency things out?
Changed more capacitors. Added  plate bypass cap to preamp.
Sounds much better now.
Parts:
- removed C?: 0.1uF, symbol Device:C
- removed J?: To VU Meter, symbol Connector:Conn_01x01_Male
- added C?: 330pF, symbol Device:C
- added R?: 270, Resistor_THT:R_Axial_DIN0516_L15.5mm_D5.0mm_P20.32mm_Horizontal, symbol Device:R
- C15: value 0.047uF -> 4.7uF
- C?: value 0.1uF -> 10uF
Connections:
- net labels added: Meter, f1, f2
- net labels removed: fl1, fl2
- wire segments 90 -> 94
Other:
- note added: "R = 740\nV = 17.7V\nI = 49mA\nP=867mW\n"
- note removed: "R = 460\nV = 15.72V\nI = 34.2mA\nP = 538mW\n\nactual current: 68mA\n"
- moved on the sheet: C?, J?, Q?, R1, R4, R?

Commit message: remove anode bypass capacitors from preamp
Parts:
- removed C?: 330pF, symbol Device:C
Connections:
- wire segments 94 -> 89
Changed lines of the file:
@@
 	5200 5200 5200 5350
 Connection ~ 5050 5200
-Wire Wire Line
-	4800 2200 4800 2250
 Connection ~ 4800 2350
 Wire Wire Line
@@
 	5800 2350 5850 2350
 Connection ~ 5800 2350
-$Comp
-L Device:C C?
-U 1 1 5FA1B98E
-P 5150 2050
-F 0 "C?" H 5265 2096 50  0000 L CNN
-F 1 "330pF" H 5265 2005 50  0000 L CNN
-F 2 "" H 5188 1900 50  0001 C CNN
-F 3 "~" H 5150 2050 50  0001 C CNN
-	1    5150 2050
-	1    0    0    -1
-$EndComp
 Wire Wire Line
 	4300 1850 4800 1850
@@
 	4800 1850 4800 1900
 Connection ~ 4300 1850
-Wire Wire Line
-	5150 1900 5150 1850
-Wire Wire Line
-	5150 1850 4800 1850
-Connection ~ 4800 1850
-Wire Wire Line
-	5150 2200 5150 2250
-Wire Wire Line
-	5150 2250 4800 2250
-Connection ~ 4800 2250
-Wire Wire Line
-	4800 2250 4800 2350
 Text HLabel 2000 2200 0    50   Input ~ 0
 f1
@@
 Text Label 2000 2350 0    50   ~ 0
 f2
+Wire Wire Line
+	4800 2200 4800 2350
 $EndSCHEMATC

Commit message: v2.5 modifications
fix the audio bleedthrough, add soft suspend switch
Parts:
- added C? (x2): 0.1uF, symbol Device:C
- added C?: 220uF, symbol Device:CP
- added RV?: 10K, symbol Device:R_POT
- added U?: LM386, symbol Amplifier_Audio:LM386
- C1, C4, C5: symbol nobsound-audio-amplifier-rescue:CP-Device -> nobsound-audio-amplifier-rescue:CP-Device-nobsound-audio-amplifier-rescue
- RV1: symbol nobsound-audio-amplifier-rescue:R_POT_Dual_Separate-Device -> nobsound-audio-amplifier-rescue:R_POT_Dual_Separate-Device-nobsound-audio-amplifier-rescue
- RV?: symbol Device:R_Potentiometer -> nobsound-audio-amplifier-rescue:R_Potentiometer-Device-nobsound-audio-amplifier-rescue
- T1: symbol local:AudioTxfmr -> nobsound-audio-amplifier-rescue:AudioTxfmr-local-nobsound-audio-amplifier-rescue
- V2: symbol local:12AX7 -> nobsound-audio-amplifier-rescue:12AX7-local-nobsound-audio-amplifier-rescue
- V3: symbol local:EL84 -> nobsound-audio-amplifier-rescue:EL84-local-nobsound-audio-amplifier-rescue
Connections:
- net labels added: GND, buffer_pwr, meter
- net labels removed: Meter
- wire segments 89 -> 103
Other:
- moved on the sheet: C15, C3, C?, J2, J3, J7, J?, Q?, R1, R13, R14, R2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

Commit message: updating schematic
Parts:
- C1, C4, C5: symbol nobsound-audio-amplifier-rescue:CP-Device-nobsound-audio-amplifier-rescue -> nobsound-audio-amplifier-rescue:CP-Device-nobsound-audio-amplifier-rescue-nobsound-audio-amplifier-rescue
- RV1: symbol nobsound-audio-amplifier-rescue:R_POT_Dual_Separate-Device-nobsound-audio-amplifier-rescue -> nobsound-audio-amplifier-rescue:R_POT_Dual_Separate-Device-nobsound-audio-amplifier-rescue-nobsound-audio-amplifier-res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
- RV?: symbol nobsound-audio-amplifier-rescue:R_Potentiometer-Device-nobsound-audio-amplifier-rescue -> nobsound-audio-amplifier-rescue:R_Potentiometer-Device-nobsound-audio-amplifier-rescue-nobsound-audio-amplifier-rescue
- T1: symbol nobsound-audio-amplifier-rescue:AudioTxfmr-local-nobsound-audio-amplifier-rescue -> nobsound-audio-amplifier-rescue:AudioTxfmr-local-nobsound-audio-amplifier-rescue-nobsound-audio-amplifier-rescue
- V2: symbol nobsound-audio-amplifier-rescue:12AX7-local-nobsound-audio-amplifier-rescue -> nobsound-audio-amplifier-rescue:12AX7-local-nobsound-audio-amplifier-rescue-nobsound-audio-amplifier-rescue
- V3: symbol nobsound-audio-amplifier-rescue:EL84-local-nobsound-audio-amplifier-rescue -> nobsound-audio-amplifier-rescue:EL84-local-nobsound-audio-amplifier-rescue-nobsound-audio-amplifier-rescue
Changed lines of the file:
@@
 $EndDescr
 $Comp
-L nobsound-audio-amplifier-rescue:AudioTxfmr-local-nobsound-audio-amplifier-rescue T?
+L nobsound-audio-amplifier-rescue:AudioTxfmr-local-nobsound-audio-amplifier-rescue-nobsound-audio-amplifier-rescue T?
 U 1 1 5F1FED34
 P 9700 5950
@@
 	9400 5650 9250 5650
 $Comp
-L nobsound-audio-amplifier-rescue:CP-Device-nobsound-audio-amplifier-rescue C?
+L nobsound-audio-amplifier-rescue:CP-Device-nobsound-audio-amplifier-rescue-nobsound-audio-amplifier-rescue C?
 U 1 1 5F1FED3C
 P 6650 5550
@@
 $EndComp
 $Comp
-L nobsound-audio-amplifier-rescue:CP-Device-nobsound-audio-amplifier-rescue C?
+L nobsound-audio-amplifier-rescue:CP-Device-nobsound-audio-amplifier-rescue-nobsound-audio-amplifier-rescue C?
 U 1 1 5F1FEDAC
 P 7550 9050
@@
 	9400 5850 9400 6200
 $Comp
-L nobsound-audio-amplifier-rescue:CP-Device-nobsound-audio-amplifier-rescue C?
+L nobsound-audio-amplifier-rescue:CP-Device-nobsound-audio-amplifier-rescue-nobsound-audio-amplifier-rescue C?
 U 1 1 5F1FEDF9
 P 9850 7650
@@
 	6000 5400 5900 5400
 $Comp
-L nobsound-audio-amplifier-rescue:EL84-local-nobsound-audio-amplifier-rescue V3
+L nobsound-audio-amplifier-rescue:EL84-local-nobsound-audio-amplifier-rescue-nobsound-audio-amplifier-rescue V3
 U 1 1 5F1E5866
 P 9400 6650
@@
 Connection ~ 9400 6200
 $Comp
-L nobsound-audio-amplifier-rescue:12AX7-local-nobsound-audio-amplifier-rescue V2
+L nobsound-audio-amplifier-rescue:12AX7-local-nobsound-audio-amplifier-rescue-nobsound-audio-amplifier-rescue V2
 U 1 1 5F1EB7D2
 P 7150 8000
@@
 	6650 7550 7150 7550
 $Comp
-L nobsound-audio-amplifier-rescue:12AX7-local-nobsound-audio-amplifier-rescue V2
+L nobsound-audio-amplifier-rescue:12AX7-local-nobsound-audio-amplifier-rescue-nobsound-audio-amplifier-rescue V2
 U 2 1 5F1F6427
 P 7150 6650
@@
 	7150 7550 7400 7550
 $Comp
-L nobsound-audio-amplifier-rescue:R_POT_Dual_Separate-Device-nobsound-audio-amplifier-rescue RV1
+L nobsound-audio-amplifier-rescue:R_POT_Dual_Separate-Device-nobsound-audio-amplifier-rescue-nobsound-audio-amplifier-rescue RV1
 U 1 1 5F23DDB3
 P 5250 8050
@@
 $EndComp
 $Comp
-L nobsound-audio-amplifier-rescue:R_Potentiometer-Device-nobsound-audio-amplifier-rescue RV?
+L nobsound-audio-amplifier-rescue:R_Potentiometer-Device-nobsound-audio-amplifier-rescue-nobsound-audio-amplifier-rescue RV?
 U 1 1 5F823B94
 P 25750 4150
