File: updated/power supply.sch (KiCad schematic (older format))
At the start: 16 parts, among them J1 Conn_IEC_Power, T2 PwrTxfmr

Commit message: finish updated schematic
Convert tables from google doc to markdown to have these in this repo
Parts:
- C17, C18, C19, C20: renamed from C?; footprint (none) -> Capacitor_THT:CP_Radial_D4.0mm_P2.00mm
- C6, C7: footprint (none) -> Capacitor_THT:CP_Radial_D10.0mm_P5.00mm
- D5, D6, D7, D8: renamed from D?; footprint (none) -> Diode_THT:D_T-1_P5.08mm_Horizontal
- R21: renamed from R?; footprint (none) -> Resistor_THT:R_Axial_DIN0516_L15.5mm_D5.0mm_P20.32mm_Horizontal
Changed lines of the file:
@@
 	4850 3800 5000 3800
 $Comp
-L power:Earth #PWR?
+L power:Earth #PWR02
 U 1 1 5F184856
 P 5800 3700
-F 0 "#PWR?" H 5800 3450 50  0001 C CNN
+F 0 "#PWR02" H 5800 3450 50  0001 C CNN
 F 1 "Earth" H 5800 3550 50  0001 C CNN
 F 2 "" H 5800 3700 50  0001 C CNN
@@
 $EndComp
 $Comp
-L power:Earth #PWR?
+L power:Earth #PWR01
 U 1 1 5F185198
 P 4000 4200
-F 0 "#PWR?" H 4000 3950 50  0001 C CNN
+F 0 "#PWR01" H 4000 3950 50  0001 C CNN
 F 1 "Earth" H 4000 4050 50  0001 C CNN
 F 2 "" H 4000 4200 50  0001 C CNN
@@
 F 0 "C6" H 6968 3991 50  0000 L CNN
 F 1 "150uF" H 6968 3900 50  0000 L CNN
-F 2 "" H 6888 3750 50  0001 C CNN
+F 2 "Capacitor_THT:CP_Radial_D10.0mm_P5.00mm" H 6888 3750 50  0001 C CNN
 F 3 "~" H 6850 3900 50  0001 C CNN
 F 4 "450V" H 6968 3809 50  0000 L CNN "Voltage"
@@
 	6850 3750 6850 3700
 $Comp
-L power:Earth #PWR?
+L power:Earth #PWR03
 U 1 1 5F18EEE6
 P 6850 4050
-F 0 "#PWR?" H 6850 3800 50  0001 C CNN
+F 0 "#PWR03" H 6850 3800 50  0001 C CNN
 F 1 "Earth" H 6850 3900 50  0001 C CNN
 F 2 "" H 6850 4050 50  0001 C CNN
@@
 F 0 "C7" H 7768 3941 50  0000 L CNN
 F 1 "150uF" H 7768 3850 50  0000 L CNN
-F 2 "" H 7688 3700 50  0001 C CNN
+F 2 "Capacitor_THT:CP_Radial_D10.0mm_P5.00mm" H 7688 3700 50  0001 C CNN
 F 3 "~" H 7650 3850 50  0001 C CNN
 F 4 "450V" H 7768 3759 50  0000 L CNN "Voltage"
@@
 	7450 3700 7650 3700
 $Comp
-L power:Earth #PWR?
+L power:Earth #PWR04
 U 1 1 5F192DBF
 P 7650 4000
-F 0 "#PWR?" H 7650 3750 50  0001 C CNN
+F 0 "#PWR04" H 7650 3750 50  0001 C CNN
 F 1 "Earth" H 7650 3850 50  0001 C CNN
 F 2 "" H 7650 4000 50  0001 C CNN
@@
 fr2
 $Comp
-L Device:D D?
+L Device:D D7
 U 1 1 5F1D3CFC
 P 5900 3900
-F 0 "D?" H 5800 3800 50  0000 C CNN
+F 0 "D7" H 5800 3800 50  0000 C CNN
 F 1 "1N4005" H 5900 3800 50  0001 C CNN
-F 2 "" H 5900 3900 50  0001 C CNN
+F 2 "Diode_THT:D_T-1_P5.08mm_Horizontal" H 5900 3900 50  0001 C CNN
 F 3 "~" H 5900 3900 50  0001 C CNN
 	1    5900 3900
@@
 $EndComp
 $Comp
-L Device:D D?
+L Device:D D5
 U 1 1 5F1DA0E8
 P 5900 3500
-F 0 "D?" H 6100 3400 50  0000 C CNN
+F 0 "D5" H 6100 3400 50  0000 C CNN
 F 1 "1N4005" H 5900 3400 50  0000 C CNN
-F 2 "" H 5900 3500 50  0001 C CNN
+F 2 "Diode_THT:D_T-1_P5.08mm_Horizontal" H 5900 3500 50  0001 C CNN
 F 3 "~" H 5900 3500 50  0001 C CNN
 	1    5900 3500
@@
 $EndComp
 $Comp
-L Device:D D?
+L Device:D D6
 U 1 1 5F1DA0F2
 P 6300 3500
-F 0 "D?" H 6400 3400 50  0000 C CNN
+F 0 "D6" H 6400 3400 50  0000 C CNN
 F 1 "1N4005" H 6300 3400 50  0001 C CNN
-F 2 "" H 6300 3500 50  0001 C CNN
+F 2 "Diode_THT:D_T-1_P5.08mm_Horizontal" H 6300 3500 50  0001 C CNN
 F 3 "~" H 6300 3500 50  0001 C CNN
 	1    6300 3500
@@
 $EndComp
 $Comp
-L Device:C C?
+L Device:C C17
 U 1 1 5F1DA0FC
 P 5900 3300
-F 0 "C?" V 5648 3300 50  0000 C CNN
+F 0 "C17" V 5648 3300 50  0000 C CNN
 F 1 "47nF" V 5739 3300 50  0000 C CNN
-F 2 "" H 5938 3150 50  0001 C CNN
+F 2 "Capacitor_THT:CP_Radial_D4.0mm_P2.00mm" H 5938 3150 50  0001 C CNN
 F 3 "~" H 5900 3300 50  0001 C CNN
 F 4 "450V" V 5900 3300 50  0001 C CNN "Voltage"
@@
 $EndComp
 $Comp
-L Device:C C?
+L Device:C C18
 U 1 1 5F1DA106
 P 6300 3300
-F 0 "C?" V 6048 3300 50  0000 C CNN
+F 0 "C18" V 6048 3300 50  0000 C CNN
 F 1 "47nF" V 6139 3300 50  0000 C CNN
-F 2 "" H 6338 3150 50  0001 C CNN
+F 2 "Capacitor_THT:CP_Radial_D4.0mm_P2.00mm" H 6338 3150 50  0001 C CNN
 F 3 "~" H 6300 3300 50  0001 C CNN
 F 4 "450V" V 6300 3300 50  0001 C CNN "Voltage"
@@
 $EndComp
 $Comp
-L Device:C C?
+L Device:C C19
 U 1 1 5F1D5EA4
 P 5900 4100
-F 0 "C?" V 5650 4100 50  0000 C CNN
+F 0 "C19" V 5650 4100 50  0000 C CNN
 F 1 "47nF" V 5739 4100 50  0000 C CNN
-F 2 "" H 5938 3950 50  0001 C CNN
+F 2 "Capacitor_THT:CP_Radial_D4.0mm_P2.00mm" H 5938 3950 50  0001 C CNN
 F 3 "~" H 5900 4100 50  0001 C CNN
 F 4 "450V" V 5900 4100 50  0001 C CNN "Voltage"
@@
 	6450 3900 6450 4100
 $Comp
-L Device:C C?
+L Device:C C20
 U 1 1 5F1D6B83
 P 6300 4100
-F 0 "C?" V 6050 4100 50  0000 C CNN
+F 0 "C20" V 6050 4100 50  0000 C CNN
 F 1 "47nF" V 6150 4100 50  0000 C CNN
-F 2 "" H 6338 3950 50  0001 C CNN
+F 2 "Capacitor_THT:CP_Radial_D4.0mm_P2.00mm" H 6338 3950 50  0001 C CNN
 F 3 "~" H 6300 4100 50  0001 C CNN
 F 4 "450V" V 6150 4300 50  0000 C CNN "Voltage"
@@
 $EndComp
 $Comp
-L Device:D D?
+L Device:D D8
 U 1 1 5F1D58F3
 P 6300 3900
-F 0 "D?" H 6400 3800 50  0000 C CNN
+F 0 "D8" H 6400 3800 50  0000 C CNN
 F 1 "1N4005" H 6300 3800 50  0001 C CNN
-F 2 "" H 6300 3900 50  0001 C CNN
+F 2 "Diode_THT:D_T-1_P5.08mm_Horizontal" H 6300 3900 50  0001 C CNN
 F 3 "~" H 6300 3900 50  0001 C CNN
 	1    6300 3900
@@
 $EndComp
 $Comp
-L Device:R R?
+L Device:R R21
 U 1 1 5F255154
 P 8150 3850
-F 0 "R?" H 8220 3941 50  0000 L CNN
+F 0 "R21" H 8220 3941 50  0000 L CNN
 F 1 "220K" H 8220 3850 50  0000 L CNN
-F 2 "" V 8080 3850 50  0001 C CNN
+F 2 "Resistor_THT:R_Axial_DIN0516_L15.5mm_D5.0mm_P20.32mm_Horizontal" V 8080 3850 50  0001 C CNN
 F 3 "~" H 8150 3850 50  0001 C CNN
 F 4 "2W" H 8220 3759 50  0000 L CNN "Power"
@@
 	8150 3700 8300 3700
 $Comp
-L power:Earth #PWR?
+L power:Earth #PWR05
 U 1 1 5F25671F
 P 8150 4000
-F 0 "#PWR?" H 8150 3750 50  0001 C CNN
+F 0 "#PWR05" H 8150 3750 50  0001 C CNN
 F 1 "Earth" H 8150 3850 50  0001 C CNN
 F 2 "" H 8150 4000 50  0001 C CNN

Commit message: adding some components to try to stop a high pitch squal sound I sometimes hear from the amp
Parts:
- added C13, C14: CP, symbol Device:CP
- added D1: D_Bridge_+AA-, symbol Device:D_Bridge_+AA-
- added U1: V7805-500, digikey-footprints:3-SIP_Module_V7805-500, symbol dk_DC-DC-Converters:V7805-500
Connections:
- net labels added: +5V, 0pv
- wire segments 36 -> 48
Changed lines of the file:
@@
 $Descr A4 11693 8268
 encoding utf-8
-Sheet 2 5
+Sheet 2 4
 Title "Nobsound Tube Amplifier Power Supply"
 Date "2020-07-20"
@@
 	1    0    0    -1
 $EndComp
+$Comp
+L dk_DC-DC-Converters:V7805-500 U1
+U 1 1 5F4F76F6
+P 8000 5050
+F 0 "U1" H 8000 5437 60  0000 C CNN
+F 1 "V7805-500" H 8000 5331 60  0000 C CNN
+F 2 "digikey-footprints:3-SIP_Module_V7805-500" H 8200 5250 60  0001 L CNN
+F 3 "https://www.cui.com/product/resource/digikeypdf/v78-500.pdf" H 8200 5350 60  0001 L CNN
+F 4 "102-1709-ND" H 8200 5450 60  0001 L CNN "Digi-Key_PN"
+F 5 "V7805-500" H 8200 5550 60  0001 L CNN "MPN"
+F 6 "Power Supplies - Board Mount" H 8200 5650 60  0001 L CNN "Category"
+F 7 "DC DC Converters" H 8200 5750 60  0001 L CNN "Family"
+F 8 "https://www.cui.com/product/resource/digikeypdf/v78-500.pdf" H 8200 5850 60  0001 L CNN "DK_Datasheet_Link"
+F 9 "/product-detail/en/cui-inc/V7805-500/102-1709-ND/1828602" H 8200 5950 60  0001 L CNN "DK_Detail_Page"
+F 10 "DC DC CONVERTER 5V 2.5W" H 8200 6050 60  0001 L CNN "Description"
+F 11 "CUI Inc." H 8200 6150 60  0001 L CNN "Manufacturer"
+F 12 "Active" H 8200 6250 60  0001 L CNN "Status"
+	1    8000 5050
+	1    0    0    -1
+$EndComp
+$Comp
+L Device:CP C13
+U 1 1 5F4FA3D7
+P 7500 5100
+F 0 "C13" H 7618 5146 50  0000 L CNN
+F 1 "CP" H 7618 5055 50  0000 L CNN
+F 2 "" H 7538 4950 50  0001 C CNN
+F 3 "~" H 7500 5100 50  0001 C CNN
+	1    7500 5100
+	1    0    0    -1
+$EndComp
+$Comp
+L Device:CP C14
+U 1 1 5F4FACD4
+P 8500 5100
+F 0 "C14" H 8618 5146 50  0000 L CNN
+F 1 "CP" H 8618 5055 50  0000 L CNN
+F 2 "" H 8538 4950 50  0001 C CNN
+F 3 "~" H 8500 5100 50  0001 C CNN
+	1    8500 5100
+	1    0    0    -1
+$EndComp
+Wire Wire Line
+	7100 4450 7100 4650
+Wire Wire Line
+	6800 4950 6750 4950
+Wire Wire Line
+	7400 4950 7500 4950
+Wire Wire Line
+	7500 4950 7600 4950
+Connection ~ 7500 4950
+Wire Wire Line
+	8400 4950 8500 4950
+Text Label 8500 4950 0    50   ~ 0
++5V
+Wire Wire Line
+	8500 5400 8500 5250
+Wire Wire Line
+	8000 5400 8000 5350
+Wire Wire Line
+	7500 5400 7500 5250
+$Comp
+L Device:D_Bridge_+AA- D1
+U 1 1 5F4F6AF1
+P 7100 4950
+F 0 "D1" H 7300 5250 50  0000 L CNN
+F 1 "D_Bridge_+AA-" H 7300 5150 50  0000 L CNN
+F 2 "" H 7100 4950 50  0001 C CNN
+F 3 "~" H 7100 4950 50  0001 C CNN
+	1    7100 4950
+	1    0    0    -1
+$EndComp
+Wire Wire Line
+	6750 5400 7500 5400
+Wire Wire Line
+	6750 4950 6750 5400
+Wire Wire Line
+	7500 5400 8000 5400
+Connection ~ 7500 5400
+Wire Wire Line
+	8000 5400 8500 5400
+Connection ~ 8000 5400
+Text Label 8500 5400 0    50   ~ 0
+0pv
 $EndSCHEMATC

Commit message: install vfd spectrograph
upgrade preamp tubes to use shielded sockets.
Parts:
- removed C14: CP, symbol Device:CP
- removed U1: V7805-500, digikey-footprints:3-SIP_Module_V7805-500, symbol dk_DC-DC-Converters:V7805-500
- added J?: VU Meter +, symbol Connector:Conn_01x01_Male
- added J?: VU Meter -, symbol Connector:Conn_01x01_Male
- added J?: VU Meter GND, symbol Connector:Conn_01x01_Male
- added PS?: IH0505D, Converter_DCDC:Converter_DCDC_XP_POWER-IHxxxxD_THT, symbol Converter_DCDC:IH0505D
Connections:
- net labels added: f1, f2
- net labels removed: +5V, 0pv
- wire segments 48 -> 49
Changed lines of the file:
@@
-$EndComp
-$Comp
-L dk_DC-DC-Converters:V7805-500 U1
-U 1 1 5F4F76F6
-P 8000 5050
-F 0 "U1" H 8000 5437 60  0000 C CNN
-F 1 "V7805-500" H 8000 5331 60  0000 C CNN
-F 2 "digikey-footprints:3-SIP_Module_V7805-500" H 8200 5250 60  0001 L CNN
-F 3 "https://www.cui.com/product/resource/digikeypdf/v78-500.pdf" H 8200 5350 60  0001 L CNN
-F 4 "102-1709-ND" H 8200 5450 60  0001 L CNN "Digi-Key_PN"
-F 5 "V7805-500" H 8200 5550 60  0001 L CNN "MPN"
-F 6 "Power Supplies - Board Mount" H 8200 5650 60  0001 L CNN "Category"
-F 7 "DC DC Converters" H 8200 5750 60  0001 L CNN "Family"
-F 8 "https://www.cui.com/product/resource/digikeypdf/v78-500.pdf" H 8200 5850 60  0001 L CNN "DK_Datasheet_Link"
-F 9 "/product-detail/en/cui-inc/V7805-500/102-1709-ND/1828602" H 8200 5950 60  0001 L CNN "DK_Detail_Page"
-F 10 "DC DC CONVERTER 5V 2.5W" H 8200 6050 60  0001 L CNN "Description"
-F 11 "CUI Inc." H 8200 6150 60  0001 L CNN "Manufacturer"
-F 12 "Active" H 8200 6250 60  0001 L CNN "Status"
-	1    8000 5050
-	1    0    0    -1
 $EndComp
 $Comp
@@
 	1    0    0    -1
 $EndComp
-$Comp
-L Device:CP C14
-U 1 1 5F4FACD4
-P 8500 5100
-F 0 "C14" H 8618 5146 50  0000 L CNN
-F 1 "CP" H 8618 5055 50  0000 L CNN
-F 2 "" H 8538 4950 50  0001 C CNN
-F 3 "~" H 8500 5100 50  0001 C CNN
-	1    8500 5100
-	1    0    0    -1
-$EndComp
 Wire Wire Line
-	7100 4450 7100 4650
+	7100 4600 7100 4650
 Wire Wire Line
 	6800 4950 6750 4950
 Wire Wire Line
 	7400 4950 7500 4950
-Wire Wire Line
-	7500 4950 7600 4950
 Connection ~ 7500 4950
-Wire Wire Line
-	8400 4950 8500 4950
-Text Label 8500 4950 0    50   ~ 0
-+5V
-Wire Wire Line
-	8500 5400 8500 5250
-Wire Wire Line
-	8000 5400 8000 5350
 Wire Wire Line
 	7500 5400 7500 5250
@@
 $EndComp
 Wire Wire Line
+	6750 4950 6750 5400
+Text Label 7100 4600 0    50   ~ 0
+f1
+Text Label 7100 5300 0    50   ~ 0
+f2
+Wire Wire Line
+	7100 5300 7100 5250
+$Comp
+L Connector:Conn_01x01_Male J?
+U 1 1 5F544D1D
+P 8950 4950
+AR Path="/5F1F04D2/5F544D1D" Ref="J?"  Part="1"
+AR Path="/5F1E3F4D/5F544D1D" Ref="J?"  Part="1"
+F 0 "J?" H 8922 4882 50  0000 R CNN
+F 1 "VU Meter +" H 8922 4973 50  0000 R CNN
+F 2 "" H 8950 4950 50  0001 C CNN
+F 3 "~" H 8950 4950 50  0001 C CNN
+	1    8950 4950
+	-1   0    0    1
+$EndComp
+$Comp
+L Connector:Conn_01x01_Male J?
+U 1 1 5F54648B
+P 8950 5050
+AR Path="/5F1F04D2/5F54648B" Ref="J?"  Part="1"
+AR Path="/5F1E3F4D/5F54648B" Ref="J?"  Part="1"
+F 0 "J?" H 8922 4982 50  0000 R CNN
+F 1 "VU Meter -" H 8922 5073 50  0000 R CNN
+F 2 "" H 8950 5050 50  0001 C CNN
+F 3 "~" H 8950 5050 50  0001 C CNN
+	1    8950 5050
+	-1   0    0    1
+$EndComp
+$Comp
+L Connector:Conn_01x01_Male J?
+U 1 1 5F54B4D4
+P 8950 5250
+AR Path="/5F1F04D2/5F54B4D4" Ref="J?"  Part="1"
+AR Path="/5F1E3F4D/5F54B4D4" Ref="J?"  Part="1"
+F 0 "J?" H 8922 5182 50  0000 R CNN
+F 1 "VU Meter GND" H 8922 5273 50  0000 R CNN
+F 2 "" H 8950 5250 50  0001 C CNN
+F 3 "~" H 8950 5250 50  0001 C CNN
+	1    8950 5250
+	-1   0    0    1
+$EndComp
+Wire Wire Line
+	8750 5350 8750 5250
+$Comp
+L power:Earth #PWR?
+U 1 1 5F54C2DF
+P 8750 5350
+F 0 "#PWR?" H 8750 5100 50  0001 C CNN
+F 1 "Earth" H 8750 5200 50  0001 C CNN
+F 2 "" H 8750 5350 50  0001 C CNN
+F 3 "~" H 8750 5350 50  0001 C CNN
+	1    8750 5350
+	1    0    0    -1
+$EndComp
+$Comp
+L Converter_DCDC:IH0505D PS?
+U 1 1 5F55887B
+P 8250 5050
+F 0 "PS?" H 8250 5417 50  0000 C CNN
+F 1 "IH0505D" H 8250 5326 50  0000 C CNN
+F 2 "Converter_DCDC:Converter_DCDC_XP_POWER-IHxxxxD_THT" H 7200 4800 50  0001 L CNN
+F 3 "https://www.xppower.com/pdfs/SF_IH.pdf" H 9300 4750 50  0001 L CNN
+	1    8250 5050
+	1    0    0    -1
+$EndComp
+Wire Wire Line
+	8750 4950 8650 4950
+Wire Wire Line
+	8750 5050 8650 5050
+Wire Wire Line
+	7500 4950 7850 4950
+Wire Wire Line
+	7850 5150 7850 5400
+Wire Wire Line
 	6750 5400 7500 5400
-Wire Wire Line
-	6750 4950 6750 5400
-Wire Wire Line
-	7500 5400 8000 5400
 Connection ~ 7500 5400
 Wire Wire Line
-	8000 5400 8500 5400
-Connection ~ 8000 5400
-Text Label 8500 5400 0    50   ~ 0
-0pv
+	7500 5400 7850 5400
 $EndSCHEMATC

Commit message: update schematic
Replaced all the counterfeit capacitor between preamp and power stage. Really opened up the sound.
Add some pictures
Parts:
- C13, C6, C7: symbol Device:CP -> nobsound-audio-amplifier-rescue:CP-Device
- J1: symbol local:Conn_IEC_Power -> nobsound-audio-amplifier-rescue:Conn_IEC_Power-local
- L1: symbol Device:L_Core_Ferrite -> nobsound-audio-amplifier-rescue:L_Core_Ferrite-Device
Other:
- note added: "364V"
Changed lines of the file:
@@
 $EndComp
 $Comp
-L local:Conn_IEC_Power J1
+L nobsound-audio-amplifier-rescue:Conn_IEC_Power-local J1
 U 1 1 5F1757DE
 P 3800 3900
@@
 	5600 3700 5800 3700
 $Comp
-L Device:L_Core_Ferrite L1
+L nobsound-audio-amplifier-rescue:L_Core_Ferrite-Device L1
 U 1 1 5F187D89
 P 7300 3700
@@
 	6850 3700 7150 3700
 $Comp
-L Device:CP C6
+L nobsound-audio-amplifier-rescue:CP-Device C6
 U 1 1 5F18A643
 P 6850 3900
+AR Path="/5F18A643" Ref="C6"  Part="1"
+AR Path="/5F1E3F4D/5F18A643" Ref="C6"  Part="1"
 F 0 "C6" H 6968 3991 50  0000 L CNN
 F 1 "150uF" H 6968 3900 50  0000 L CNN
@@
 $EndComp
 $Comp
-L Device:CP C7
+L nobsound-audio-amplifier-rescue:CP-Device C7
 U 1 1 5F1901A9
 P 7650 3850
+AR Path="/5F1901A9" Ref="C7"  Part="1"
+AR Path="/5F1E3F4D/5F1901A9" Ref="C7"  Part="1"
 F 0 "C7" H 7768 3941 50  0000 L CNN
 F 1 "150uF" H 7768 3850 50  0000 L CNN
@@
 $EndComp
 $Comp
-L Device:CP C13
+L nobsound-audio-amplifier-rescue:CP-Device C13
 U 1 1 5F4FA3D7
 P 7500 5100
+AR Path="/5F4FA3D7" Ref="C13"  Part="1"
+AR Path="/5F1E3F4D/5F4FA3D7" Ref="C13"  Part="1"
 F 0 "C13" H 7618 5146 50  0000 L CNN
 F 1 "CP" H 7618 5055 50  0000 L CNN
@@
 Wire Wire Line
 	7500 5400 7850 5400
+Text Notes 8050 3500 0    50   ~ 0
+364V
 $EndSCHEMATC

Commit message: It didn't sound right to me
I don't understand how changing the cathode bypass a bit made the amp a lot more brighter. Theory is the power supply was over loaded before and it was not able to drive the high frequency things out?
Changed more capacitors. Added  plate bypass cap to preamp.
Sounds much better now.
Parts:
- removed J?: VU Meter +, symbol Connector:Conn_01x01_Male
- removed J?: VU Meter -, symbol Connector:Conn_01x01_Male
- removed J?: VU Meter GND, symbol Connector:Conn_01x01_Male
Connections:
- net labels added: meter_gnd, meter_pwr
- no-connect marks 0 -> 2
Changed lines of the file:
@@
 	7650 3700 8150 3700
 Connection ~ 7650 3700
-Text Label 8300 3700 0    50   ~ 0
-B+
-Text Label 5600 4400 2    50   ~ 0
-fl1
-Text Label 5600 4500 2    50   ~ 0
-fl2
-Text Label 5600 4700 2    50   ~ 0
-fr1
-Text Label 5600 4800 2    50   ~ 0
-fr2
 $Comp
 L Device:D D7
@@
 	7100 5300 7100 5250
 $Comp
-L Connector:Conn_01x01_Male J?
-U 1 1 5F544D1D
-P 8950 4950
-AR Path="/5F1F04D2/5F544D1D" Ref="J?"  Part="1"
-AR Path="/5F1E3F4D/5F544D1D" Ref="J?"  Part="1"
-F 0 "J?" H 8922 4882 50  0000 R CNN
-F 1 "VU Meter +" H 8922 4973 50  0000 R CNN
-F 2 "" H 8950 4950 50  0001 C CNN
-F 3 "~" H 8950 4950 50  0001 C CNN
-	1    8950 4950
-	-1   0    0    1
-$EndComp
-$Comp
-L Connector:Conn_01x01_Male J?
-U 1 1 5F54648B
-P 8950 5050
-AR Path="/5F1F04D2/5F54648B" Ref="J?"  Part="1"
-AR Path="/5F1E3F4D/5F54648B" Ref="J?"  Part="1"
-F 0 "J?" H 8922 4982 50  0000 R CNN
-F 1 "VU Meter -" H 8922 5073 50  0000 R CNN
-F 2 "" H 8950 5050 50  0001 C CNN
-F 3 "~" H 8950 5050 50  0001 C CNN
-	1    8950 5050
-	-1   0    0    1
-$EndComp
-$Comp
-L Connector:Conn_01x01_Male J?
-U 1 1 5F54B4D4
-P 8950 5250
-AR Path="/5F1F04D2/5F54B4D4" Ref="J?"  Part="1"
-AR Path="/5F1E3F4D/5F54B4D4" Ref="J?"  Part="1"
-F 0 "J?" H 8922 5182 50  0000 R CNN
-F 1 "VU Meter GND" H 8922 5273 50  0000 R CNN
-F 2 "" H 8950 5250 50  0001 C CNN
-F 3 "~" H 8950 5250 50  0001 C CNN
-	1    8950 5250
-	-1   0    0    1
-$EndComp
-Wire Wire Line
-	8750 5350 8750 5250
-$Comp
 L power:Earth #PWR?
 U 1 1 5F54C2DF
@@
 Text Notes 8050 3500 0    50   ~ 0
 364V
+Text HLabel 8300 3700 2    50   Output ~ 0
+B+
+NoConn ~ 5600 4100
+NoConn ~ 5600 4200
+Text HLabel 5600 4400 2    50   Output ~ 0
+fl1
+Text HLabel 5600 4500 2    50   Output ~ 0
+fl2
+Text HLabel 5600 4700 2    50   Output ~ 0
+fr1
+Text HLabel 5600 4800 2    50   Output ~ 0
+fr2
+Wire Wire Line
+	8750 5050 8750 5350
+Text HLabel 8750 4950 2    50   Output ~ 0
+meter_pwr
+Text HLabel 8750 5050 2    50   Output ~ 0
+meter_gnd
 $EndSCHEMATC

Commit message: v2.5 modifications
fix the audio bleedthrough, add soft suspend switch
Parts:
- removed C13: CP, symbol nobsound-audio-amplifier-rescue:CP-Device
- removed D1: D_Bridge_+AA-, symbol Device:D_Bridge_+AA-
- removed PS?: IH0505D, Converter_DCDC:Converter_DCDC_XP_POWER-IHxxxxD_THT, symbol Converter_DCDC:IH0505D
- C6, C7: symbol nobsound-audio-amplifier-rescue:CP-Device -> nobsound-audio-amplifier-rescue:CP-Device-nobsound-audio-amplifier-rescue
- J1: symbol nobsound-audio-amplifier-rescue:Conn_IEC_Power-local -> nobsound-audio-amplifier-rescue:Conn_IEC_Power-local-nobsound-audio-amplifier-rescue
- L1: symbol nobsound-audio-amplifier-rescue:L_Core_Ferrite-Device -> nobsound-audio-amplifier-rescue:L_Core_Ferrite-Device-nobsound-audio-amplifier-rescue
- S1: symbol local:SW_SPST -> nobsound-audio-amplifier-rescue:SW_SPST-local-nobsound-audio-amplifier-rescue
- T2: symbol local:PwrTxfmr -> nobsound-audio-amplifier-rescue:PwrTxfmr-local-nobsound-audio-amplifier-rescue
Connections:
- net labels removed: f1, f2, meter_gnd, meter_pwr
- wire segments 49 -> 36
Other:
- note added: "390V"
- note removed: "364V"
Changed lines of the file:
@@
 $Descr A4 11693 8268
 encoding utf-8
-Sheet 2 4
+Sheet 2 6
 Title "Nobsound Tube Amplifier Power Supply"
 Date "2020-07-20"
@@
 $EndDescr
 $Comp
-L local:PwrTxfmr T2
+L nobsound-audio-amplifier-rescue:PwrTxfmr-local-nobsound-audio-amplifier-rescue T2
 U 1 1 5F15D5D5
 P 5300 4100
@@
 $EndComp
 $Comp
-L local:SW_SPST S1
+L nobsound-audio-amplifier-rescue:SW_SPST-local-nobsound-audio-amplifier-rescue S1
 U 1 1 5F164E42
 P 4600 3800
@@
 $EndComp
 $Comp
-L nobsound-audio-amplifier-rescue:Conn_IEC_Power-local J1
+L nobsound-audio-amplifier-rescue:Conn_IEC_Power-local-nobsound-audio-amplifier-rescue J1
 U 1 1 5F1757DE
 P 3800 3900
@@
 	5600 3700 5800 3700
 $Comp
-L nobsound-audio-amplifier-rescue:L_Core_Ferrite-Device L1
+L nobsound-audio-amplifier-rescue:L_Core_Ferrite-Device-nobsound-audio-amplifier-rescue L1
 U 1 1 5F187D89
 P 7300 3700
@@
 	6850 3700 7150 3700
 $Comp
-L nobsound-audio-amplifier-rescue:CP-Device C6
+L nobsound-audio-amplifier-rescue:CP-Device-nobsound-audio-amplifier-rescue C6
 U 1 1 5F18A643
 P 6850 3900
@@
 $EndComp
 $Comp
-L nobsound-audio-amplifier-rescue:CP-Device C7
+L nobsound-audio-amplifier-rescue:CP-Device-nobsound-audio-amplifier-rescue C7
 U 1 1 5F1901A9
 P 7650 3850
@@
 	1    0    0    -1
 $EndComp
-$Comp
-L nobsound-audio-amplifier-rescue:CP-Device C13
-U 1 1 5F4FA3D7
-P 7500 5100
-AR Path="/5F4FA3D7" Ref="C13"  Part="1"
-AR Path="/5F1E3F4D/5F4FA3D7" Ref="C13"  Part="1"
-F 0 "C13" H 7618 5146 50  0000 L CNN
-F 1 "CP" H 7618 5055 50  0000 L CNN
-F 2 "" H 7538 4950 50  0001 C CNN
-F 3 "~" H 7500 5100 50  0001 C CNN
-	1    7500 5100
-	1    0    0    -1
-$EndComp
-Wire Wire Line
-	7100 4600 7100 4650
-Wire Wire Line
-	6800 4950 6750 4950
-Wire Wire Line
-	7400 4950 7500 4950
-Connection ~ 7500 4950
-Wire Wire Line
-	7500 5400 7500 5250
-$Comp
-L Device:D_Bridge_+AA- D1
-U 1 1 5F4F6AF1
-P 7100 4950
-F 0 "D1" H 7300 5250 50  0000 L CNN
-F 1 "D_Bridge_+AA-" H 7300 5150 50  0000 L CNN
-F 2 "" H 7100 4950 50  0001 C CNN
-F 3 "~" H 7100 4950 50  0001 C CNN
-	1    7100 4950
-	1    0    0    -1
-$EndComp
-Wire Wire Line
-	6750 4950 6750 5400
-Text Label 7100 4600 0    50   ~ 0
-f1
-Text Label 7100 5300 0    50   ~ 0
-f2
-Wire Wire Line
-	7100 5300 7100 5250
-$Comp
-L power:Earth #PWR?
-U 1 1 5F54C2DF
-P 8750 5350
-F 0 "#PWR?" H 8750 5100 50  0001 C CNN
-F 1 "Earth" H 8750 5200 50  0001 C CNN
-F 2 "" H 8750 5350 50  0001 C CNN
-F 3 "~" H 8750 5350 50  0001 C CNN
-	1    8750 5350
-	1    0    0    -1
-$EndComp
-$Comp
-L Converter_DCDC:IH0505D PS?
-U 1 1 5F55887B
-P 8250 5050
-F 0 "PS?" H 8250 5417 50  0000 C CNN
-F 1 "IH0505D" H 8250 5326 50  0000 C CNN
-F 2 "Converter_DCDC:Converter_DCDC_XP_POWER-IHxxxxD_THT" H 7200 4800 50  0001 L CNN
-F 3 "https://www.xppower.com/pdfs/SF_IH.pdf" H 9300 4750 50  0001 L CNN
-	1    8250 5050
-	1    0    0    -1
-$EndComp
-Wire Wire Line
-	8750 4950 8650 4950
-Wire Wire Line
-	8750 5050 8650 5050
-Wire Wire Line
-	7500 4950 7850 4950
-Wire Wire Line
-	7850 5150 7850 5400
-Wire Wire Line
-	6750 5400 7500 5400
-Connection ~ 7500 5400
-Wire Wire Line
-	7500 5400 7850 5400
 Text Notes 8050 3500 0    50   ~ 0
-364V
+390V
 Text HLabel 8300 3700 2    50   Output ~ 0
 B+
@@
 Text HLabel 5600 4800 2    50   Output ~ 0
 fr2
-Wire Wire Line
-	8750 5050 8750 5350
-Text HLabel 8750 4950 2    50   Output ~ 0
-meter_pwr
-Text HLabel 8750 5050 2    50   Output ~ 0
-meter_gnd
 $EndSCHEMATC
