File: updated/power supply.sch (KiCad schematic (older format))
At the start: 16 parts, among them J1 Conn_IEC_Power, T2 PwrTxfmr

Commit message: updating schematic
Parts:
- C6, C7: symbol nobsound-audio-amplifier-rescue:CP-Device-nobsound-audio-amplifier-rescue -> nobsound-audio-amplifier-rescue:CP-Device-nobsound-audio-amplifier-rescue-nobsound-audio-amplifier-rescue
- J1: symbol nobsound-audio-amplifier-rescue:Conn_IEC_Power-local-nobsound-audio-amplifier-rescue -> nobsound-audio-amplifier-rescue:Conn_IEC_Power-local-nobsound-audio-amplifier-rescue-nobsound-audio-amplifier-rescue
- L1: symbol nobsound-audio-amplifier-rescue:L_Core_Ferrite-Device-nobsound-audio-amplifier-rescue -> nobsound-audio-amplifier-rescue:L_Core_Ferrite-Device-nobsound-audio-amplifier-rescue-nobsound-audio-amplifier-rescue
- S1: symbol nobsound-audio-amplifier-rescue:SW_SPST-local-nobsound-audio-amplifier-rescue -> nobsound-audio-amplifier-rescue:SW_SPST-local-nobsound-audio-amplifier-rescue-nobsound-audio-amplifier-rescue
- T2: symbol nobsound-audio-amplifier-rescue:PwrTxfmr-local-nobsound-audio-amplifier-rescue -> nobsound-audio-amplifier-rescue:PwrTxfmr-local-nobsound-audio-amplifier-rescue-nobsound-audio-amplifier-rescue
Other:
- note added: "Just powering filaments:\nInput 120V, 0.1A (12W)\n* measured with fluke clamp meter, \n not likely accurate, we can't have less power in than out"
- note added: "Unloaded voltage: 7.34V\nI of 4 tubes: 2.34A\nLoaded voltage: 6.97V\nso about 16 W"
Changed lines of the file:
@@
 $Descr A4 11693 8268
 encoding utf-8
-Sheet 2 6
+Sheet 6 6
 Title "Nobsound Tube Amplifier Power Supply"
 Date "2020-07-20"
@@
 $EndDescr
 $Comp
-L nobsound-audio-amplifier-rescue:PwrTxfmr-local-nobsound-audio-amplifier-rescue T2
+L nobsound-audio-amplifier-rescue:PwrTxfmr-local-nobsound-audio-amplifier-rescue-nobsound-audio-amplifier-rescue T2
 U 1 1 5F15D5D5
 P 5300 4100
@@
 $EndComp
 $Comp
-L nobsound-audio-amplifier-rescue:SW_SPST-local-nobsound-audio-amplifier-rescue S1
+L nobsound-audio-amplifier-rescue:SW_SPST-local-nobsound-audio-amplifier-rescue-nobsound-audio-amplifier-rescue S1
 U 1 1 5F164E42
 P 4600 3800
@@
 $EndComp
 $Comp
-L nobsound-audio-amplifier-rescue:Conn_IEC_Power-local-nobsound-audio-amplifier-rescue J1
+L nobsound-audio-amplifier-rescue:Conn_IEC_Power-local-nobsound-audio-amplifier-rescue-nobsound-audio-amplifier-rescue J1
 U 1 1 5F1757DE
 P 3800 3900
@@
 	5600 3700 5800 3700
 $Comp
-L nobsound-audio-amplifier-rescue:L_Core_Ferrite-Device-nobsound-audio-amplifier-rescue L1
+L nobsound-audio-amplifier-rescue:L_Core_Ferrite-Device-nobsound-audio-amplifier-rescue-nobsound-audio-amplifier-rescue L1
 U 1 1 5F187D89
 P 7300 3700
@@
 	6850 3700 7150 3700
 $Comp
-L nobsound-audio-amplifier-rescue:CP-Device-nobsound-audio-amplifier-rescue C6
+L nobsound-audio-amplifier-rescue:CP-Device-nobsound-audio-amplifier-rescue-nobsound-audio-amplifier-rescue C6
 U 1 1 5F18A643
 P 6850 3900
@@
 $EndComp
 $Comp
-L nobsound-audio-amplifier-rescue:CP-Device-nobsound-audio-amplifier-rescue C7
+L nobsound-audio-amplifier-rescue:CP-Device-nobsound-audio-amplifier-rescue-nobsound-audio-amplifier-rescue C7
 U 1 1 5F1901A9
 P 7650 3850
@@
 Text HLabel 5600 4800 2    50   Output ~ 0
 fr2
+Text Notes 5850 5050 0    50   ~ 0
+Unloaded voltage: 7.34V\nI of 4 tubes: 2.34A\nLoaded voltage: 6.97V\nso about 16 W
+Text Notes 3300 5300 0    50   ~ 0
+Just powering filaments:\nInput 120V, 0.1A  (12W)\n* measured with fluke clamp meter, \n  not likely accurate, we can't have less power in than out
 $EndSCHEMATC
