File: updated/vfd.sch (KiCad schematic (older format))
At the start: 5 parts

Commit message: updating schematic
Parts:
- C? (x2): symbol nobsound-audio-amplifier-rescue:CP-Device-nobsound-audio-amplifier-rescue -> nobsound-audio-amplifier-rescue:CP-Device-nobsound-audio-amplifier-rescue-nobsound-audio-amplifier-rescue
Changed lines of the file:
@@
 $EndComp
 $Comp
-L nobsound-audio-amplifier-rescue:CP-Device-nobsound-audio-amplifier-rescue C?
+L nobsound-audio-amplifier-rescue:CP-Device-nobsound-audio-amplifier-rescue-nobsound-audio-amplifier-rescue C?
 U 1 1 60AF9688
 P 1700 1350
@@
 $EndComp
 $Comp
-L nobsound-audio-amplifier-rescue:CP-Device-nobsound-audio-amplifier-rescue C?
+L nobsound-audio-amplifier-rescue:CP-Device-nobsound-audio-amplifier-rescue-nobsound-audio-amplifier-rescue C?
 U 1 1 60B90348
 P 1800 3500
